File: pcb.kicad_sch (KiCad schematic)
At the start: 0 parts

Commit message: Removing pads and adding more TPs and also mounting holes
Parts:
- added H1, H2, H3, H7: MountingHole, MountingHole:MountingHole_3.2mm_M3_DIN965_Pad, symbol Mechanical:MountingHole
Other:
- note added: "Board outline"
