File: housekeeping.kicad_sch (KiCad schematic)
At the start: 8 parts, among them U18 LMR43620MSC5RPERQ1

Commit message: Fixing circuit errors
Parts:
- U18: footprint _Power_Board:RPE0009A-MFG -> _PowerBoard:RPE0009A-MFG
Changed lines of the file:
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@@
 			)
 		)
-		(property "Footprint" "_Power_Board:RPE0009A-MFG"
+		(property "Footprint" "_PowerBoard:RPE0009A-MFG"
 			(at 105.41 85.09 0)
 			(effects
