File: housekeeping.kicad_sch (KiCad schematic)
At the start: 8 parts, among them U18 LMR43620MSC5RPERQ1

Commit message: Completing layout
Parts:
- renumbered C80 to C79, C81 to C80, C82 to C81, C83 to C82, C84 to C83, C85 to C84, U18 to U17
