File: power_sns.kicad_sch (KiCad schematic)
At the start: 2 parts, among them U2 PINA745AIRELR

Commit message: Adding control stuff
Parts:
- C17: footprint Capacitor_SMD:C_1206_3216Metric -> Capacitor_SMD:C_0603_1608Metric; Mfr Murata Electronics -> KYOCERA AVX; Mfr P/N GCM31C5C1H104FA16L -> 06035C104K4T2A; Supplier_1 P/N 490-GCM31C5C1H104FA16LTR-ND -> 478-KAM15AR71H104KTTR-ND; Supplier_1 Unit Price 0.98000 -> 0.10000
Connections:
- net +5V: now also C17.2; no longer C17.1
- net GND: now also C17.1; no longer C17.2

Commit message: Adding in connections to schematic
Parts:
- U2: footprint REL0014A_PINA745AIRELR_TEX -> _Power_Board:REL0014A_PINA745AIRELR_TEX

Commit message: Working on layout now
Parts:
- U7: renamed from U2; Mfr (none) -> Texas Instruments; Mfr P/N (none) -> INA745AIRELR; Supplier_1 (none) -> Texas Instruments; Supplier_1 P/N (none) -> 1; Supplier_1 Price @ Qty (none) -> 1; Supplier_1 Unit Price (none) -> 2.044
- renumbered C17 to C44
Changed lines of the file:
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@@
 		(on_board yes)
 		(dnp no)
-		(property "Reference" "#PWR015"
+		(property "Reference" "#PWR054"
 			(at 119.38 81.28 0)
 			(effects
@@
 			(project "PowerBoard"
 				(path "/99785679-20de-4827-b4cc-bc3c187068c9/9564929a-642e-4163-88c2-45054b63a5ed/3068c1f6-122c-49ae-9c21-f8ebc0263ff5"
-					(reference "#PWR015")
+					(reference "#PWR054")
 					(unit 1)
 				)
 				(path "/99785679-20de-4827-b4cc-bc3c187068c9/9564929a-642e-4163-88c2-45054b63a5ed/f48ac83e-9a77-49aa-aabc-f4682142862d"
-					(reference "#PWR016")
+					(reference "#PWR078")
 					(unit 1)
 				)
@@
 		(dnp no)
 		(fields_autoplaced yes)
-		(property "Reference" "#PWR019"
+		(property "Reference" "#PWR053"
 			(at 102.87 97.79 0)
 			(effects
@@
 			(project "PowerBoard"
 				(path "/99785679-20de-4827-b4cc-bc3c187068c9/9564929a-642e-4163-88c2-45054b63a5ed/3068c1f6-122c-49ae-9c21-f8ebc0263ff5"
-					(reference "#PWR019")
+					(reference "#PWR053")
 					(unit 1)
 				)
 				(path "/99785679-20de-4827-b4cc-bc3c187068c9/9564929a-642e-4163-88c2-45054b63a5ed/f48ac83e-9a77-49aa-aabc-f4682142862d"
-					(reference "#PWR020")
+					(reference "#PWR077")
 					(unit 1)
 				)
@@
 		(on_board yes)
 		(dnp no)
-		(property "Reference" "U2"
+		(property "Reference" "U7"
 			(at 149.86 66.04 0)
 			(effects
@@
 			)
 		)
-		(property "Description" ""
-			(at 170.18 76.2 0)
-			(effects
-				(font
-					(size 1.27 1.27)
-				)
-				(hide yes)
-			)
-		)
-		(property "Mfr" ""
-			(at 170.18 76.2 0)
-			(effects
-				(font
-					(size 1.27 1.27)
-				)
-				(hide yes)
-			)
-		)
-		(property "Mfr P/N" ""
-			(at 170.18 76.2 0)
-			(effects
-				(font
-					(size 1.27 1.27)
-				)
-				(hide yes)
-			)
-		)
-		(property "Supplier_1" ""
-			(at 170.18 76.2 0)
-			(effects
-				(font
-					(size 1.27 1.27)
-				)
-				(hide yes)
-			)
-		)
-		(property "Supplier_1 P/N" ""
-			(at 170.18 76.2 0)
-			(effects
-				(font
-					(size 1.27 1.27)
-				)
-				(hide yes)
-			)
-		)
-		(property "Supplier_1 Unit Price" ""
-			(at 170.18 76.2 0)
-			(effects
-				(font
-					(size 1.27 1.27)
-				)
-				(hide yes)
-			)
-		)
-		(property "Supplier_1 Price @ Qty" ""
+		(property "Description" "40V, 16BIT HIGH-PRECISION I2C OU"
+			(at 170.18 76.2 0)
+			(effects
+				(font
+					(size 1.27 1.27)
+				)
+				(hide yes)
+			)
+		)
+		(property "Mfr" "Texas Instruments"
+			(at 170.18 76.2 0)
+			(effects
+				(font
+					(size 1.27 1.27)
+				)
+				(hide yes)
+			)
+		)
+		(property "Mfr P/N" "INA745AIRELR"
+			(at 170.18 76.2 0)
+			(effects
+				(font
+					(size 1.27 1.27)
+				)
+				(hide yes)
+			)
+		)
+		(property "Supplier_1" "Texas Instruments"
+			(at 170.18 76.2 0)
+			(effects
+				(font
+					(size 1.27 1.27)
+				)
+				(hide yes)
+			)
+		)
+		(property "Supplier_1 P/N" "1"
+			(at 170.18 76.2 0)
+			(effects
+				(font
+					(size 1.27 1.27)
+				)
+				(hide yes)
+			)
+		)
+		(property "Supplier_1 Unit Price" "2.044"
+			(at 170.18 76.2 0)
+			(effects
+				(font
+					(size 1.27 1.27)
+				)
+				(hide yes)
+			)
+		)
+		(property "Supplier_1 Price @ Qty" "1"
 			(at 170.18 76.2 0)
 			(effects
@@
 			(project "PowerBoard"
 				(path "/99785679-20de-4827-b4cc-bc3c187068c9/9564929a-642e-4163-88c2-45054b63a5ed/3068c1f6-122c-49ae-9c21-f8ebc0263ff5"
-					(reference "U2")
+					(reference "U7")
 					(unit 1)
 				)
 				(path "/99785679-20de-4827-b4cc-bc3c187068c9/9564929a-642e-4163-88c2-45054b63a5ed/f48ac83e-9a77-49aa-aabc-f4682142862d"
-					(reference "U3")
+					(reference "U11")
 					(unit 1)
 				)
@@
 		(on_board yes)
 		(dnp no)
-		(property "Reference" "#PWR017"
+		(property "Reference" "#PWR055"
 			(at 191.77 81.28 0)
 			(effects
@@
 			(project "PowerBoard"
 				(path "/99785679-20de-4827-b4cc-bc3c187068c9/9564929a-642e-4163-88c2-45054b63a5ed/3068c1f6-122c-49ae-9c21-f8ebc0263ff5"
-					(reference "#PWR017")
+					(reference "#PWR055")
 					(unit 1)
 				)
 				(path "/99785679-20de-4827-b4cc-bc3c187068c9/9564929a-642e-4163-88c2-45054b63a5ed/f48ac83e-9a77-49aa-aabc-f4682142862d"
-					(reference "#PWR018")
+					(reference "#PWR079")
 					(unit 1)
 				)
@@
 		(on_board yes)
 		(dnp no)
-		(property "Reference" "C17"
+		(property "Reference" "C44"
 			(at 98.552 88.392 0)
 			(effects
@@
 			(project "PowerBoard"
 				(path "/99785679-20de-4827-b4cc-bc3c187068c9/9564929a-642e-4163-88c2-45054b63a5ed/3068c1f6-122c-49ae-9c21-f8ebc0263ff5"
-					(reference "C17")
+					(reference "C44")
 					(unit 1)
 				)
 				(path "/99785679-20de-4827-b4cc-bc3c187068c9/9564929a-642e-4163-88c2-45054b63a5ed/f48ac83e-9a77-49aa-aabc-f4682142862d"
-					(reference "C18")
+					(reference "C55")
 					(unit 1)
 				)
@@
 		(dnp no)
 		(fields_autoplaced yes)
-		(property "Reference" "#PWR013"
+		(property "Reference" "#PWR052"
 			(at 99.06 83.82 0)
 			(effects
@@
 			(project "PowerBoard"
 				(path "/99785679-20de-4827-b4cc-bc3c187068c9/9564929a-642e-4163-88c2-45054b63a5ed/3068c1f6-122c-49ae-9c21-f8ebc0263ff5"
-					(reference "#PWR013")
+					(reference "#PWR052")
 					(unit 1)
 				)
 				(path "/99785679-20de-4827-b4cc-bc3c187068c9/9564929a-642e-4163-88c2-45054b63a5ed/f48ac83e-9a77-49aa-aabc-f4682142862d"
-					(reference "#PWR014")
-					(unit 1)
-				)
+					(reference "#PWR076")
+					(unit 1)
+				)

Commit message: Working on layout for dev board
Other:
- note added: "INA745 Block Diagram"
- note added: "INA745 I2C Select"
Changed lines of the file:
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@@
 		(members "SDA" "SCL")
+	)
+	(text "INA745 Block Diagram"
+		(exclude_from_sim no)
+		(at 30.48 146.558 0)
+		(effects
+			(font
+				(size 1.27 1.27)
+				(thickness 0.254)
+				(bold yes)
+			)
+		)
+	)
+	(text "INA745 I2C Select"
+		(exclude_from_sim no)
+		(at 108.966 146.812 0)
+		(effects
+			(font
+				(size 1.27 1.27)
+				(thickness 0.254)
+				(bold yes)
+			)
+		)
 	)
 	(junction

Commit message: Fixing circuit errors
Parts:
- U7: footprint _Power_Board:REL0014A_PINA745AIRELR_TEX -> _PowerBoard:REL0014A_PINA745AIRELR_TEX
Changed lines of the file:
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@@
 			)
 		)
-		(property "Footprint" "_Power_Board:REL0014A_PINA745AIRELR_TEX"
+		(property "Footprint" "_PowerBoard:REL0014A_PINA745AIRELR_TEX"
 			(at 170.18 76.2 0)
 			(effects

Commit message: Completing layout
Parts:
- renumbered C44 to C43, U7 to U6
