File: mcu.kicad_sch (KiCad schematic)
At the start: 30 parts, among them J1 Conn_01x02_Socket, U3 RP2350A, X1 ABM8-272-T3

Commit message: Powerboard planning layout
Parts:
- C19, C20, C21, C22, C23, C24, C27, C28, C29, C30, C31, C32, C33, C34: footprint Capacitor_SMD:C_0402_1005Metric -> Capacitor_SMD:C_0603_1608Metric
- C25, C26: footprint Resistor_SMD:R_0201_0603Metric -> Capacitor_SMD:C_0603_1608Metric
- R10, R11, R13, R16, R9: footprint Resistor_SMD:R_0402_1005Metric -> Resistor_SMD:R_0603_1608Metric
- R12, R14, R15, R7, R8: footprint Resistor_SMD:R_0201_0603Metric -> Resistor_SMD:R_0603_1608Metric
- U3: footprint _BMS:QFN-60_7X7_RPI -> _PowerBoard:QFN-60_7X7_RPI
- X1: footprint _BMS:ABM8-272-T3_ABR -> _PowerBoard:ABM8-272-T3_ABR
Changed lines of the file:
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@@
 			)
 		)
-		(property "Footprint" "Capacitor_SMD:C_0402_1005Metric"
+		(property "Footprint" "Capacitor_SMD:C_0603_1608Metric"
 			(at 90.17 83.5152 0)
 			(effects
@@
 			)
 		)
-		(property "Datasheet" "https://search.murata.co.jp/Ceramy/image/img/A01X/G101/ENG/GRM155C71H104JE19-01A.pdf"
+		(property "Datasheet" "~"
 			(at 93.98 82.55 0)
 			(effects
@@
 			)
 		)
-		(property "Description" "CAP CER 0.1UF 50V X7S 0402"
+		(property "Description" "Unpolarized capacitor"
 			(at 93.98 82.55 0)
 			(effects
@@
 			)
 		)
-		(property "Footprint" "Resistor_SMD:R_0201_0603Metric"
+		(property "Footprint" "Capacitor_SMD:C_0603_1608Metric"
 			(at 169.8752 175.26 0)
 			(effects
@@
 			)
 		)
-		(property "Footprint" "Capacitor_SMD:C_0402_1005Metric"
+		(property "Footprint" "Capacitor_SMD:C_0603_1608Metric"
 			(at 235.2548 113.03 0)
 			(effects
@@
 			)
 		)
-		(property "Footprint" "Resistor_SMD:R_0402_1005Metric"
+		(property "Footprint" "Resistor_SMD:R_0603_1608Metric"
 			(at 212.09 34.798 90)
 			(effects
@@
 			)
 		)
-		(property "Datasheet" "https://www.koaspeer.com/pdfs/RK73-RT.pdf"
+		(property "Datasheet" "~"
 			(at 212.09 33.02 0)
 			(effects
@@
 			)
 		)
-		(property "Description" "RES 1K OHM 1% 1/10W 0402"
+		(property "Description" "Resistor"
 			(at 212.09 33.02 0)
 			(effects
@@
 			)
 		)
-		(property "Footprint" "Resistor_SMD:R_0201_0603Metric"
+		(property "Footprint" "Resistor_SMD:R_0603_1608Metric"
 			(at 167.132 158.75 90)
 			(effects
@@
 			)
 		)
-		(property "Footprint" "Resistor_SMD:R_0201_0603Metric"
+		(property "Footprint" "Resistor_SMD:R_0603_1608Metric"
 			(at 54.61 111.252 90)
 			(effects
@@
 			)
 		)
-		(property "Footprint" "Resistor_SMD:R_0402_1005Metric"
+		(property "Footprint" "Resistor_SMD:R_0603_1608Metric"
 			(at 72.39 122.428 90)
 			(effects
@@
 			)
 		)
-		(property "Footprint" "Capacitor_SMD:C_0402_1005Metric"
+		(property "Footprint" "Capacitor_SMD:C_0603_1608Metric"
 			(at 90.17 70.8152 0)
 			(effects
@@
 			)
 		)
-		(property "Datasheet" "https://search.murata.co.jp/Ceramy/image/img/A01X/G101/ENG/GRM155C71H104JE19-01A.pdf"
+		(property "Datasheet" "~"
 			(at 93.98 69.85 0)
 			(effects
@@
 			)
 		)
-		(property "Description" "CAP CER 0.1UF 50V X7S 0402"
+		(property "Description" "Unpolarized capacitor"
 			(at 93.98 69.85 0)
 			(effects
@@
 			)
 		)
-		(property "Footprint" "Capacitor_SMD:C_0402_1005Metric"
+		(property "Footprint" "Capacitor_SMD:C_0603_1608Metric"
 			(at 90.17 113.9952 0)
 			(effects
@@
 			)
 		)
-		(property "Datasheet" "https://search.murata.co.jp/Ceramy/image/img/A01X/G101/ENG/GRM155C71H104JE19-01A.pdf"
+		(property "Datasheet" "~"
 			(at 93.98 113.03 0)
 			(effects
@@
 			)
 		)
-		(property "Description" "CAP CER 0.1UF 50V X7S 0402"
+		(property "Description" "Unpolarized capacitor"
 			(at 93.98 113.03 0)
 			(effects
@@
 			)
 		)
-		(property "Footprint" "Capacitor_SMD:C_0402_1005Metric"
+		(property "Footprint" "Capacitor_SMD:C_0603_1608Metric"
 			(at 90.17 106.3752 0)
 			(effects
@@
 			)
 		)
-		(property "Datasheet" "https://search.murata.co.jp/Ceramy/image/img/A01X/G101/ENG/GRM155C71H104JE19-01A.pdf"
+		(property "Datasheet" "~"
 			(at 93.98 105.41 0)
 			(effects
@@
 			)
 		)
-		(property "Description" "CAP CER 0.1UF 50V X7S 0402"
+		(property "Description" "Unpolarized capacitor"
 			(at 93.98 105.41 0)
 			(effects
@@
 			)
 		)
-		(property "Footprint" "Capacitor_SMD:C_0402_1005Metric"
+		(property "Footprint" "Capacitor_SMD:C_0603_1608Metric"
 			(at 267.97 99.3648 0)
 			(effects
@@
 			)
 		)
-		(property "Datasheet" "https://search.murata.co.jp/Ceramy/image/img/A01X/G101/ENG/GRM155R60J475ME87-01.pdf"
+		(property "Datasheet" "~"
 			(at 264.16 100.33 0)
 			(effects
@@
 			)
 		)
-		(property "Description" "CAP CER 4.7UF 6.3V X5R 0402"
+		(property "Description" "Unpolarized capacitor"
 			(at 264.16 100.33 0)
 			(effects
@@
 			)
 		)
-		(property "Footprint" "Capacitor_SMD:C_0402_1005Metric"
+		(property "Footprint" "Capacitor_SMD:C_0603_1608Metric"
 			(at 223.2152 129.54 0)
 			(effects
@@
 			)
 		)
-		(property "Footprint" "Resistor_SMD:R_0402_1005Metric"
+		(property "Footprint" "Resistor_SMD:R_0603_1608Metric"
 			(at 248.412 107.95 90)
 			(effects
@@
 			)
 		)
-		(property "Footprint" "Capacitor_SMD:C_0402_1005Metric"
+		(property "Footprint" "Capacitor_SMD:C_0603_1608Metric"
 			(at 208.5848 130.81 0)
 			(effects
@@
 			)
 		)
-		(property "Footprint" "Capacitor_SMD:C_0402_1005Metric"
+		(property "Footprint" "Capacitor_SMD:C_0603_1608Metric"
 			(at 195.8848 130.81 0)
 			(effects
@@
 			)
 		)
-		(property "Footprint" "Capacitor_SMD:C_0402_1005Metric"
+		(property "Footprint" "Capacitor_SMD:C_0603_1608Metric"
 			(at 267.97 91.7448 0)
 			(effects
@@
 			)
 		)
-		(property "Footprint" "Capacitor_SMD:C_0402_1005Metric"
+		(property "Footprint" "Capacitor_SMD:C_0603_1608Metric"
 			(at 211.1248 49.53 0)
 			(effects
@@
 			)
 		)
-		(property "Datasheet" "https://search.murata.co.jp/Ceramy/image/img/A01X/G101/ENG/GRM155C71H104JE19-01A.pdf"
+		(property "Datasheet" "~"
 			(at 212.09 53.34 0)
 			(effects
@@
 			)
 		)
-		(property "Description" "CAP CER 0.1UF 50V X7S 0402"
+		(property "Description" "Unpolarized capacitor"
 			(at 212.09 53.34 0)
 			(effects
@@
 			)
 		)
-		(property "Footprint" "_BMS:QFN-60_7X7_RPI"
+		(property "Footprint" "_PowerBoard:QFN-60_7X7_RPI"
 			(at 115.57 57.15 0)
 			(effects
@@
 			)
 		)
-		(property "Footprint" "Resistor_SMD:R_0201_0603Metric"
+		(property "Footprint" "Resistor_SMD:R_0603_1608Metric"
 			(at 223.52 66.548 90)
 			(effects
@@
 			)
 		)
-		(property "Footprint" "Capacitor_SMD:C_0402_1005Metric"
+		(property "Footprint" "Capacitor_SMD:C_0603_1608Metric"
 			(at 90.17 58.1152 0)
 			(effects
@@
 			)
 		)
-		(property "Datasheet" "https://search.murata.co.jp/Ceramy/image/img/A01X/G101/ENG/GRM155C71H104JE19-01A.pdf"
+		(property "Datasheet" "~"
 			(at 93.98 57.15 0)
 			(effects
@@
 			)
 		)
-		(property "Description" "CAP CER 0.1UF 50V X7S 0402"
+		(property "Description" "Unpolarized capacitor"
 			(at 93.98 57.15 0)
 			(effects
@@
 			)
 		)
-		(property "Footprint" "Resistor_SMD:R_0201_0603Metric"
+		(property "Footprint" "Resistor_SMD:R_0603_1608Metric"
 			(at 223.52 69.088 90)
 			(effects
@@
 			)
 		)
-		(property "Footprint" "_BMS:ABM8-272-T3_ABR"
+		(property "Footprint" "_PowerBoard:ABM8-272-T3_ABR"
 			(at 132.08 163.83 0)
 			(effects
@@
 			)
 		)
-		(property "Footprint" "Resistor_SMD:R_0201_0603Metric"
+		(property "Footprint" "Resistor_SMD:R_0603_1608Metric"
 			(at 54.61 109.728 90)
 			(effects
@@
 			)
 		)
-		(property "Footprint" "Resistor_SMD:R_0201_0603Metric"
+		(property "Footprint" "Capacitor_SMD:C_0603_1608Metric"
 			(at 124.1552 175.26 0)
 			(effects
@@
 			)
 		)
-		(property "Footprint" "Capacitor_SMD:C_0402_1005Metric"
+		(property "Footprint" "Capacitor_SMD:C_0603_1608Metric"
 			(at 90.17 131.7752 0)
 			(effects
@@
 			)
 		)
-		(property "Datasheet" "https://search.murata.co.jp/Ceramy/image/img/A01X/G101/ENG/GRM155C71H104JE19-01A.pdf"
+		(property "Datasheet" "~"
 			(at 93.98 130.81 0)
 			(effects
@@
 			)
 		)
-		(property "Description" "CAP CER 0.1UF 50V X7S 0402"
+		(property "Description" "Unpolarized capacitor"
 			(at 93.98 130.81 0)
 			(effects
@@
 			)
 		)
-		(property "Footprint" "Resistor_SMD:R_0402_1005Metric"
+		(property "Footprint" "Resistor_SMD:R_0603_1608Metric"
 			(at 64.77 30.988 90)
 			(effects
@@
 			)
 		)
-		(property "Datasheet" "https://www.koaspeer.com/pdfs/RN73R.pdf"
+		(property "Datasheet" "~"
 			(at 64.77 29.21 0)
 			(effects
@@
 			)
 		)
-		(property "Description" "RES 33K OHM 0.1% 1/16W 0402"
+		(property "Description" "Resistor"
 			(at 64.77 29.21 0)
 			(effects
@@
 			)
 		)
-		(property "Footprint" "Resistor_SMD:R_0402_1005Metric"
+		(property "Footprint" "Resistor_SMD:R_0603_1608Metric"
 			(at 64.77 31.242 90)
 			(effects
@@
 			)
 		)
-		(property "Datasheet" "https://www.koaspeer.com/pdfs/RN73R.pdf"
+		(property "Datasheet" "~"
 			(at 64.77 33.02 0)
 			(effects
@@
 			)
 		)
-		(property "Description" "RES 33K OHM 0.1% 1/16W 0402"
+		(property "Description" "Resistor"
 			(at 64.77 33.02 0)
 			(effects
@@
 			)
 		)
-		(property "Footprint" "Capacitor_SMD:C_0402_1005Metric"
+		(property "Footprint" "Capacitor_SMD:C_0603_1608Metric"
 			(at 251.1552 120.65 0)
 			(effects
