File: boost_in_sns.kicad_sch (KiCad schematic)
At the start: 2 parts, among them U2 PINA745AIRELR

Commit message: BOM in folder
Parts:
- C17: JLCPCB Status (none) -> JLC in-stock package match; Mfr P/N GCM31C5C1H104FA16L -> CL31B104KBCNNNC; Supplier_1 Digikey -> LCSC; Supplier_1 P/N 490-GCM31C5C1H104FA16LTR-ND -> C24497; Supplier_1 Unit Price 0.98000 -> (none)
Changed lines of the file:
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@@
 			)
 		)
-		(property "Mfr P/N" "GCM31C5C1H104FA16L"
+		(property "Mfr P/N" "CL31B104KBCNNNC"
 			(at 102.87 87.63 0)
 			(effects
@@
 			)
 		)
-		(property "Supplier_1" "Digikey"
+		(property "Supplier_1" "LCSC"
 			(at 102.87 87.63 0)
 			(effects
@@
 			)
 		)
-		(property "Supplier_1 P/N" "490-GCM31C5C1H104FA16LTR-ND"
+		(property "Supplier_1 P/N" "C24497"
 			(at 102.87 87.63 0)
 			(effects
@@
 			)
 		)
-		(property "Supplier_1 Unit Price" "0.98000"
+		(property "Supplier_1 Unit Price" ""
 			(at 102.87 87.63 0)
 			(effects
@@
 			(at 102.87 87.63 0)
 			(effects
+				(font
+					(size 1.27 1.27)
+				)
+				(hide yes)
+			)
+		)
+		(property "JLCPCB Status" "JLC in-stock package match"
+			(at 102.87 87.63 0)
+			(effects
