File: boost_load_sw.kicad_sch (KiCad schematic)
At the start: 33 parts, among them Q2 PSMN020-100YS, U14 TPS16851VMAR, U9 LM5050-1

Commit message: BOM in folder
Parts:
- C23: JLCPCB Status (none) -> JLC in-stock package match; Mfr P/N GCM21B5C1H223FA16L -> CL21B223KBANNNC; Supplier_1 Digikey -> LCSC; Supplier_1 P/N 490-GCM21B5C1H223FA16LTR-ND -> C1729; Supplier_1 Unit Price 0.52000 -> (none)
- C29: JLCPCB Status (none) -> JLC in-stock package match; Mfr P/N 08055C104J4T2A -> CC0805KRX7R9BB104; Supplier_1 Digikey -> LCSC; Supplier_1 P/N 478-KAM21BR71H104JTTR-ND -> C49678; Supplier_1 Unit Price 0.18000 -> (none)
- C34: JLCPCB Status (none) -> JLC in-stock package match; Mfr P/N GCM1885C2A471FA16D -> 0603B472K500NT; Supplier_1 Digikey -> LCSC; Supplier_1 P/N 490-GCM1885C2A471FA16DTR-ND -> C53987; Supplier_1 Unit Price 0.16000 -> (none)
- C41: JLCPCB Status (none) -> JLC in-stock package match; Mfr P/N C0603C221F5GACAUTO -> CL10B224KA8NNNC; Supplier_1 Digikey -> LCSC; Supplier_1 P/N 399-C0603C221F5GACAUTOTR-ND -> C21120; Supplier_1 Unit Price 0.85000 -> (none)
- C46, C56: Supplier_1 Digikey -> LCSC; Supplier_1 P/N 490-GCM1885C2A101FA16DTR-ND -> C527967; Supplier_1 Unit Price 0.14000 -> (none)
- C51: JLCPCB Status (none) -> JLC in-stock package match; Mfr P/N GCM1885C2A220FA16D -> CL10C220JB8NNNC; Supplier_1 Digikey -> LCSC; Supplier_1 P/N 490-16413-2-ND -> C1653; Supplier_1 Unit Price 0.14000 -> (none)
- C61: JLCPCB Status (none) -> JLC in-stock package match; Mfr P/N GCM1885C2A100FA16D -> CL10C100JB8NNNC; Supplier_1 Digikey -> LCSC; Supplier_1 P/N 490-GCM1885C2A100FA16DTR-ND -> C1634; Supplier_1 Unit Price 0.14000 -> (none)
- D12, D2: Supplier_1 Digikey -> LCSC; Supplier_1 P/N 1727-7326-2-ND -> C549269; Supplier_1 Unit Price 1 -> (none)
- D17, D7: JLCPCB Status (none) -> Similar JLC in-stock package match; Mfr P/N TPSMB28CA-VR -> SMBJ28CA; Supplier_1 Digikey -> LCSC; Supplier_1 P/N TPSMB28CA-VRTR-ND -> C353369; Supplier_1 Unit Price 0.23000 -> (none)
- Q2: Supplier_1 Digikey -> LCSC; Supplier_1 P/N 1727-4286-2-ND -> C89867; Supplier_1 Unit Price 1.42000 -> (none)
- R14, R31: JLCPCB Status (none) -> JLC in-stock package match; Mfr P/N RNCF0603BKC1M00 -> 0603WAF1004T5E; Supplier_1 Digikey -> LCSC; Supplier_1 P/N RNCF0603BKC1M00TR-ND -> C22935; Supplier_1 Unit Price 0.11000 -> (none)
- R30: Supplier_1 Digikey -> LCSC; Supplier_1 P/N P36KDBTR-ND -> C473249; Supplier_1 Unit Price 0.10000 -> (none)
- R32: Supplier_1 Digikey -> LCSC; Supplier_1 P/N 2019-RN73R1JTTD6732B25TR-ND -> C2506885; Supplier_1 Unit Price 0.12000 -> (none)
- R33: JLCPCB Status (none) -> Similar JLC in-stock package match; Mfr P/N ERA-3AEB151V -> RC0603JR-07150RL; Supplier_1 Digikey -> LCSC; Supplier_1 P/N P150DBTR-ND -> C126805; Supplier_1 Unit Price 0.10000 -> (none)
- R35: Supplier_1 Digikey -> LCSC; Supplier_1 P/N 2019-RN73R1JTTD1261B25TR-ND -> C2508249; Supplier_1 Unit Price 0.12000 -> (none)
- R40: JLCPCB Status (none) -> Similar JLC in-stock package match; Mfr P/N ERA-3AEB4640V -> FRC0603F4642TS; Supplier_1 Digikey -> LCSC; Supplier_1 P/N 10-ERA-3AEB4640VTR-ND -> C3013203; Supplier_1 Unit Price 0.10000 -> (none)
- R45: JLCPCB Status (none) -> JLC in-stock package match; Mfr P/N ERA-3AEB103V -> 0603WAF1001T5E; Supplier_1 Digikey -> LCSC; Supplier_1 P/N P10KDBTR-ND -> C21190; Supplier_1 Unit Price 0.10000 -> (none)
- R50, R55: JLCPCB Status (none) -> JLC in-stock package match; Mfr P/N ERA-3AEB333V -> 0603WAF3302T5E; Supplier_1 Digikey -> LCSC; Supplier_1 P/N P33KDBTR-ND -> C4216; Supplier_1 Unit Price 0.10000 -> (none)
- R6: JLCPCB Status (none) -> JLC in-stock package match; Mfr P/N ERA-3AEB101V -> RC0603FR-07100RL; Supplier_1 Digikey -> LCSC; Supplier_1 P/N P100DBTR-ND -> C105588; Supplier_1 Unit Price 0.10000 -> (none)
- R60: Supplier_1 Digikey -> LCSC; Supplier_1 P/N RTAN1206BKE10R0TR-ND -> C346735; Supplier_1 Unit Price 0.42000 -> (none)
- R65: JLCPCB Status (none) -> JLC in-stock package match; Mfr P/N ERA-3AEB244V -> 0603WAF2403T5E; Supplier_1 Digikey -> LCSC; Supplier_1 P/N P240KDBTR-ND -> C4197; Supplier_1 Unit Price 0.10000 -> (none)
- U14: Supplier_1 Texas Instruments -> LCSC; Supplier_1 P/N TPS16851VMAR -> C48705346; Supplier_1 Unit Price 10.32 -> (none)
- U9: JLCPCB Status (none) -> JLC in-stock package match; Mfr P/N (none) -> LM5050MKX-1/NOPB; Supplier_1 (none) -> LCSC; Supplier_1 P/N (none) -> C473393
