File: buck_converter.kicad_sch (KiCad schematic)
At the start: 19 parts, among them U19 LT8640SEV_PBF

Commit message: BOM in folder
Parts:
- 5V_HK2: Supplier_1 Digikey -> LCSC; Supplier_1 P/N 952-1478-2-ND -> C3345122; Supplier_1 Unit Price 0.28000 -> (none)
- C100, C98, C99: JLCPCB Status (none) -> Similar JLC in-stock package match; Mfr P/N CL32B106KBJNNWE -> CS3225X7R106K500NRL; Supplier_1 DigiKey -> LCSC; Supplier_1 P/N 1276-3388-2-ND -> C2918502; Supplier_1 Unit Price $0.22 -> (none)
- C101, C102: JLCPCB Status (none) -> JLC in-stock package match; Mfr P/N UMK107AB7105KA-T -> CL10A105KB8NNNC; Supplier_1 DigiKey -> LCSC; Supplier_1 P/N 587-3247-2-ND -> C15849; Supplier_1 Unit Price $0.08 -> (none)
- C103: Supplier_1 DigiKey -> LCSC; Supplier_1 P/N 1276-1009-2-ND -> C5137477; Supplier_1 Unit Price $0.08 -> (none)
- C104: Supplier_1 DigiKey -> LCSC; Supplier_1 P/N 1276-1000-2-ND -> C1591; Supplier_1 Unit Price $0.08 -> (none)
- C105: JLCPCB Status (none) -> JLC in-stock package match; Mfr P/N (none) -> CL10A105KB8NNNC; Supplier_1 DigiKey -> LCSC; Supplier_1 P/N 587-3247-2-ND -> C15849; Supplier_1 Unit Price $0.08 -> (none)
- C106: JLCPCB Status (none) -> JLC in-stock package match; Mfr P/N GRM1885C1H4R7CA01D -> 0603CG4R7C500NT; Supplier_1 DigiKey -> LCSC; Supplier_1 P/N 490-12722-2-ND -> C1669; Supplier_1 Unit Price 0.12 -> (none)
- C107: Supplier_1 DigiKey -> LCSC; Supplier_1 P/N 1276-3376-2-ND -> C2932477; Supplier_1 Unit Price $0.68 -> (none)
- D13: Supplier_1 Digikey -> LCSC; Supplier_1 P/N SMCJ26ALFTR-ND -> C152085; Supplier_1 Unit Price 0.35000 -> (none)
- D14: Supplier_1 DigiKey -> LCSC; Supplier_1 P/N 4878-SMF5.0ATR-ND -> C151296; Supplier_1 Unit Price 0.25000 -> (none)
- FB6: Supplier_1 DigiKey -> LCSC; Supplier_1 P/N 732-3431-2-ND -> C5155961; Supplier_1 Unit Price $0.68 -> (none)
- L6: Supplier_1 Digikey -> LCSC; Supplier_1 P/N 240-TYA40201R5M-10TR-ND -> C2649052; Supplier_1 Unit Price 0.37000 -> (none)
- R47: Supplier_1 Digikey -> LCSC; Supplier_1 P/N P18.2KDBTR-ND -> C527967; Supplier_1 Unit Price 0.10000 -> (none)
- R48: JLCPCB Status (none) -> JLC in-stock package match; Mfr P/N ERJ-3EKF1004V -> 0603WAF1004T5E; Supplier_1 DigiKey -> LCSC; Supplier_1 P/N P1.00MHTR-ND -> C22935; Supplier_1 Unit Price 0.10 -> (none)
- R54: JLCPCB Status (none) -> JLC in-stock package match; Mfr P/N ERA-3AEB2433V -> 0603WAF2433T5E; Supplier_1 DigiKey -> LCSC; Supplier_1 P/N P243KDBTR-ND -> C23351; Supplier_1 Unit Price 0.10 -> (none)
- U19: Supplier_1 Digikey -> LCSC; Supplier_1 P/N 505-LT8640SEV#PBF-ND -> C514429; Supplier_1 Unit Price 13.52000 -> (none)
