File: ldo.kicad_sch (KiCad schematic)
At the start: 5 parts, among them U17 TLV75533PDBV

Commit message: BOM in folder
Parts:
- 3V3_HK2: Supplier_1 Digikey -> LCSC; Supplier_1 P/N 952-1478-2-ND -> C3345122; Supplier_1 Unit Price 0.28000 -> (none)
- C96, C97: JLCPCB Status (none) -> JLC in-stock package match; Mfr P/N (none) -> CL10A105KB8NNNC; Supplier_1 DigiKey -> LCSC; Supplier_1 P/N 587-3247-2-ND -> C15849; Supplier_1 Unit Price $0.08 -> (none)
- D12: Supplier_1 Digikey -> LCSC; Supplier_1 P/N F7701TR-ND -> C2649858; Supplier_1 Unit Price 0.49000 -> (none)
- U17: Supplier_1 Digikey -> LCSC; Supplier_1 P/N 296-50411-2-ND -> C404027; Supplier_1 Unit Price 0.36000 -> (none)
Changed lines of the file:
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@@
 			)
 		)
-		(property "Supplier_1" "Digikey"
-			(at 177.8 86.36 0)
-			(effects
-				(font
-					(size 1.27 1.27)
-				)
-				(hide yes)
-			)
-		)
-		(property "Supplier_1 P/N" "952-1478-2-ND"
-			(at 177.8 86.36 0)
-			(effects
-				(font
-					(size 1.27 1.27)
-				)
-				(hide yes)
-			)
-		)
-		(property "Supplier_1 Unit Price" "0.28000"
+		(property "Supplier_1" "LCSC"
+			(at 177.8 86.36 0)
+			(effects
+				(font
+					(size 1.27 1.27)
+				)
+				(hide yes)
+			)
+		)
+		(property "Supplier_1 P/N" "C3345122"
+			(at 177.8 86.36 0)
+			(effects
+				(font
+					(size 1.27 1.27)
+				)
+				(hide yes)
+			)
+		)
+		(property "Supplier_1 Unit Price" ""
 			(at 177.8 86.36 0)
 			(effects
@@
 			)
 		)
-		(property "Supplier_1" "Digikey"
+		(property "Supplier_1" "LCSC"
 			(at 175.26 96.52 0)
 			(effects
@@
 			)
 		)
-		(property "Supplier_1 P/N" "F7701TR-ND"
+		(property "Supplier_1 P/N" "C2649858"
 			(at 175.26 96.52 0)
 			(effects
@@
 			)
 		)
-		(property "Supplier_1 Unit Price" "0.49000"
+		(property "Supplier_1 Unit Price" ""
 			(at 175.26 96.52 0)
 			(effects
@@
 			)
 		)
-		(property "Supplier_1" "DigiKey"
-			(at 162.56 96.52 0)
-			(effects
-				(font
-					(size 1.27 1.27)
-				)
-				(hide yes)
-			)
-		)
-		(property "Supplier_1 P/N" "587-3247-2-ND"
-			(at 162.56 96.52 0)
-			(effects
-				(font
-					(size 1.27 1.27)
-				)
-				(hide yes)
-			)
-		)
-		(property "Supplier_1 Unit Price" "$0.08"
+		(property "Supplier_1" "LCSC"
+			(at 162.56 96.52 0)
+			(effects
+				(font
+					(size 1.27 1.27)
+				)
+				(hide yes)
+			)
+		)
+		(property "Supplier_1 P/N" "C15849"
+			(at 162.56 96.52 0)
+			(effects
+				(font
+					(size 1.27 1.27)
+				)
+				(hide yes)
+			)
+		)
+		(property "Supplier_1 Unit Price" ""
 			(at 162.56 96.52 0)
 			(effects
@@
 		)
 		(property "Unit" ""
+			(at 162.56 96.52 0)
+			(effects
+				(font
+					(size 1.27 1.27)
+				)
+				(hide yes)
+			)
+		)
+		(property "Mfr P/N" "CL10A105KB8NNNC"
+			(at 162.56 96.52 0)
+			(effects
+				(font
+					(size 1.27 1.27)
+				)
+				(hide yes)
+			)
+		)
+		(property "JLCPCB Status" "JLC in-stock package match"
 			(at 162.56 96.52 0)
 			(effects
@@
 			)
 		)
-		(property "Supplier_1" "DigiKey"
-			(at 127 96.52 0)
-			(effects
-				(font
-					(size 1.27 1.27)
-				)
-				(hide yes)
-			)
-		)
-		(property "Supplier_1 P/N" "587-3247-2-ND"
-			(at 127 96.52 0)
-			(effects
-				(font
-					(size 1.27 1.27)
-				)
-				(hide yes)
-			)
-		)
-		(property "Supplier_1 Unit Price" "$0.08"
+		(property "Supplier_1" "LCSC"
+			(at 127 96.52 0)
+			(effects
+				(font
+					(size 1.27 1.27)
+				)
+				(hide yes)
+			)
+		)
+		(property "Supplier_1 P/N" "C15849"
+			(at 127 96.52 0)
+			(effects
+				(font
+					(size 1.27 1.27)
+				)
+				(hide yes)
+			)
+		)
+		(property "Supplier_1 Unit Price" ""
 			(at 127 96.52 0)
 			(effects
@@
 		)
 		(property "Unit" ""
+			(at 127 96.52 0)
+			(effects
+				(font
+					(size 1.27 1.27)
+				)
+				(hide yes)
+			)
+		)
+		(property "Mfr P/N" "CL10A105KB8NNNC"
+			(at 127 96.52 0)
+			(effects
+				(font
+					(size 1.27 1.27)
+				)
+				(hide yes)
+			)
+		)
+		(property "JLCPCB Status" "JLC in-stock package match"
 			(at 127 96.52 0)
 			(effects
@@
 			)
 		)
-		(property "Supplier_1" "Digikey"
+		(property "Supplier_1" "LCSC"
 			(at 151.13 93.98 0)
 			(effects
@@
 			)
 		)
-		(property "Supplier_1 P/N" "296-50411-2-ND"
+		(property "Supplier_1 P/N" "C404027"
 			(at 151.13 93.98 0)
 			(effects
@@
 			)
 		)
-		(property "Supplier_1 Unit Price" "0.36000"
+		(property "Supplier_1 Unit Price" ""
 			(at 151.13 93.98 0)
 			(effects
