File: navlight_load_sw2.kicad_sch (KiCad schematic)
At the start: 6 parts, among them U14 TPS26400PWP

Commit message: BOM in folder
Parts:
- C75: JLCPCB Status (none) -> JLC in-stock package match; Mfr P/N UMK107AB7105KA-T -> CL10A105KB8NNNC; Supplier_1 DigiKey -> LCSC; Supplier_1 P/N UMK107AB7105KA-T -> C15849; Supplier_1 Unit Price $0.08 -> (none)
- C76: Supplier_1 DigiKey -> LCSC; Supplier_1 P/N 1276-1000-2-ND -> C1591; Supplier_1 Unit Price $0.08 -> (none)
- FLT_HK2, TP2: Supplier_1 Digikey -> LCSC; Supplier_1 P/N 952-1478-2-ND -> C3345122; Supplier_1 Unit Price 0.28000 -> (none)
- R50: JLCPCB Status (none) -> JLC in-stock package match; Mfr P/N ERA-3AEB8061V -> 0603WAF8061T5E; Supplier_1 DigiKey -> LCSC; Supplier_1 P/N P8.06KDBTR-ND -> C23112; Supplier_1 Unit Price 0.10 -> (none)
- U14: Supplier_1 Digikey -> LCSC; Supplier_1 P/N 296-TPS26400PWPRTR-ND -> C3662862; Supplier_1 Unit Price 2.85000 -> (none)
Changed lines of the file:
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@@
 			)
 		)
-		(property "Supplier_1" "Digikey"
+		(property "Supplier_1" "LCSC"
 			(at 152.4 114.3 0)
 			(effects
@@
 			)
 		)
-		(property "Supplier_1 P/N" "952-1478-2-ND"
+		(property "Supplier_1 P/N" "C3345122"
 			(at 152.4 114.3 0)
 			(effects
@@
 			)
 		)
-		(property "Supplier_1 Unit Price" "0.28000"
+		(property "Supplier_1 Unit Price" ""
 			(at 152.4 114.3 0)
 			(effects
@@
 			)
 		)
-		(property "Supplier_1" "DigiKey"
-			(at 165.1 100.33 0)
-			(effects
-				(font
-					(size 1.27 1.27)
-				)
-				(hide yes)
-			)
-		)
-		(property "Supplier_1 P/N" "1276-1000-2-ND"
-			(at 165.1 100.33 0)
-			(effects
-				(font
-					(size 1.27 1.27)
-				)
-				(hide yes)
-			)
-		)
-		(property "Supplier_1 Unit Price" "$0.08"
+		(property "Supplier_1" "LCSC"
+			(at 165.1 100.33 0)
+			(effects
+				(font
+					(size 1.27 1.27)
+				)
+				(hide yes)
+			)
+		)
+		(property "Supplier_1 P/N" "C1591"
+			(at 165.1 100.33 0)
+			(effects
+				(font
+					(size 1.27 1.27)
+				)
+				(hide yes)
+			)
+		)
+		(property "Supplier_1 Unit Price" ""
 			(at 165.1 100.33 0)
 			(effects
@@
 			)
 		)
-		(property "Mfr P/N" "ERA-3AEB8061V"
-			(at 175.26 100.33 0)
-			(effects
-				(font
-					(size 1.27 1.27)
-				)
-				(hide yes)
-			)
-		)
-		(property "Supplier_1" "DigiKey"
-			(at 175.26 100.33 0)
-			(effects
-				(font
-					(size 1.27 1.27)
-				)
-				(hide yes)
-			)
-		)
-		(property "Supplier_1 P/N" "P8.06KDBTR-ND"
-			(at 175.26 100.33 0)
-			(effects
-				(font
-					(size 1.27 1.27)
-				)
-				(hide yes)
-			)
-		)
-		(property "Supplier_1 Unit Price" "0.10"
+		(property "Mfr P/N" "0603WAF8061T5E"
+			(at 175.26 100.33 0)
+			(effects
+				(font
+					(size 1.27 1.27)
+				)
+				(hide yes)
+			)
+		)
+		(property "Supplier_1" "LCSC"
+			(at 175.26 100.33 0)
+			(effects
+				(font
+					(size 1.27 1.27)
+				)
+				(hide yes)
+			)
+		)
+		(property "Supplier_1 P/N" "C23112"
+			(at 175.26 100.33 0)
+			(effects
+				(font
+					(size 1.27 1.27)
+				)
+				(hide yes)
+			)
+		)
+		(property "Supplier_1 Unit Price" ""
 			(at 175.26 100.33 0)
 			(effects
@@
 		)
 		(property "Unit" ""
+			(at 175.26 100.33 0)
+			(effects
+				(font
+					(size 1.27 1.27)
+				)
+				(hide yes)
+			)
+		)
+		(property "JLCPCB Status" "JLC in-stock package match"
 			(at 175.26 100.33 0)
 			(effects
@@
 			)
 		)
-		(property "Supplier_1" "Digikey"
-			(at 170.18 82.55 0)
-			(effects
-				(font
-					(size 1.27 1.27)
-				)
-				(hide yes)
-			)
-		)
-		(property "Supplier_1 P/N" "952-1478-2-ND"
-			(at 170.18 82.55 0)
-			(effects
-				(font
-					(size 1.27 1.27)
-				)
-				(hide yes)
-			)
-		)
-		(property "Supplier_1 Unit Price" "0.28000"
+		(property "Supplier_1" "LCSC"
+			(at 170.18 82.55 0)
+			(effects
+				(font
+					(size 1.27 1.27)
+				)
+				(hide yes)
+			)
+		)
+		(property "Supplier_1 P/N" "C3345122"
+			(at 170.18 82.55 0)
+			(effects
+				(font
+					(size 1.27 1.27)
+				)
+				(hide yes)
+			)
+		)
+		(property "Supplier_1 Unit Price" ""
 			(at 170.18 82.55 0)
 			(effects
@@
 			)
 		)
-		(property "Mfr P/N" "UMK107AB7105KA-T"
-			(at 123.19 73.66 0)
-			(effects
-				(font
-					(size 1.27 1.27)
-				)
-				(hide yes)
-			)
-		)
-		(property "Supplier_1" "DigiKey"
-			(at 123.19 73.66 0)
-			(effects
-				(font
-					(size 1.27 1.27)
-				)
-				(hide yes)
-			)
-		)
-		(property "Supplier_1 P/N" "UMK107AB7105KA-T"
-			(at 123.19 73.66 0)
-			(effects
-				(font
-					(size 1.27 1.27)
-				)
-				(hide yes)
-			)
-		)
-		(property "Supplier_1 Unit Price" "$0.08"
+		(property "Mfr P/N" "CL10A105KB8NNNC"
+			(at 123.19 73.66 0)
+			(effects
+				(font
+					(size 1.27 1.27)
+				)
+				(hide yes)
+			)
+		)
+		(property "Supplier_1" "LCSC"
+			(at 123.19 73.66 0)
+			(effects
+				(font
+					(size 1.27 1.27)
+				)
+				(hide yes)
+			)
+		)
+		(property "Supplier_1 P/N" "C15849"
+			(at 123.19 73.66 0)
+			(effects
+				(font
+					(size 1.27 1.27)
+				)
+				(hide yes)
+			)
+		)
+		(property "Supplier_1 Unit Price" ""
 			(at 123.19 73.66 0)
 			(effects
@@
 		)
 		(property "Supplier_2 Price @ Qty" ""
+			(at 123.19 73.66 0)
+			(effects
+				(font
+					(size 1.27 1.27)
+				)
+				(hide yes)
+			)
+		)
+		(property "JLCPCB Status" "JLC in-stock package match"
 			(at 123.19 73.66 0)
 			(effects
@@
 			)
 		)
-		(property "Supplier_1" "Digikey"
+		(property "Supplier_1" "LCSC"
 			(at 152.4 82.55 0)
 			(effects
@@
 			)
 		)
-		(property "Supplier_1 P/N" "296-TPS26400PWPRTR-ND"
+		(property "Supplier_1 P/N" "C3662862"
 			(at 152.4 82.55 0)
 			(effects
@@
 			)
 		)
-		(property "Supplier_1 Unit Price" "2.85000"
+		(property "Supplier_1 Unit Price" ""
 			(at 152.4 82.55 0)
 			(effects
