File: output.kicad_sch (KiCad schematic)
At the start: 20 parts, among them U12 TLV75533PDBV, U13 LT8640SEV_PBF

Commit message: Schematic updates
Parts:
- R45: Mfr Panasonic Electronic Components -> UNI-ROYAL(Uniroyal Elec); Mfr P/N ERA-3AEB1822V -> 0603WAF1822T5E; Supplier_1 P/N C22793 -> C22892
Changed lines of the file:
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@@
 			)
 		)
+		(property "Supplier_1 Price @ Qty" ""
+			(at 232.41 63.5 0)
+			(effects
+				(font
+					(size 1.27 1.27)
+				)
+				(hide yes)
+			)
+		)
+		(property "Supplier_2 Price @ Qty" ""
+			(at 232.41 63.5 0)
+			(effects
+				(font
+					(size 1.27 1.27)
+				)
+				(hide yes)
+			)
+		)
 		(pin "1"
 		)
@@
 			)
 		)
+		(property "Supplier_1 Price @ Qty" ""
+			(at 107.95 95.25 0)
+			(effects
+				(font
+					(size 1.27 1.27)
+				)
+				(hide yes)
+			)
+		)
+		(property "Supplier_2 Price @ Qty" ""
+			(at 107.95 95.25 0)
+			(effects
+				(font
+					(size 1.27 1.27)
+				)
+				(hide yes)
+			)
+		)
 		(pin "1"
 		)
@@
 			)
 		)
+		(property "Supplier_1 Price @ Qty" ""
+			(at 209.55 66.04 0)
+			(effects
+				(font
+					(size 1.27 1.27)
+				)
+				(hide yes)
+			)
+		)
+		(property "Supplier_2 Price @ Qty" ""
+			(at 209.55 66.04 0)
+			(effects
+				(font
+					(size 1.27 1.27)
+				)
+				(hide yes)
+			)
+		)
 		(pin "2"
 		)
@@
 			)
 		)
-		(property "Datasheet" "https://industrial.panasonic.com/cdbs/www-data/pdf/RDM0000/AOA0000C307.pdf"
+		(property "Datasheet" "https://jlcpcb.com/api/file/downloadByFileSystemAccessId/8586178083586392065"
 			(at 95.25 95.25 0)
 			(effects
@@
 			)
 		)
-		(property "Description" "18.2 kOhms ±0.1% 0.1W, 1/10W Chip Resistor 0603 (1608 Metric) Automotive AEC-Q200 Thin Film"
+		(property "Description" "100mW 18.2kΩ 75V Thick Film Resistor ±1% ±100ppm/℃ 0603"
 			(at 95.25 95.25 0)
 			(effects
@@
 			)
 		)
-		(property "Mfr" "Panasonic Electronic Components"
+		(property "Mfr" "UNI-ROYAL(Uniroyal Elec)"
 			(at 95.25 95.25 0)
 			(effects
@@
 			)
 		)
-		(property "Mfr P/N" "ERA-3AEB1822V"
+		(property "Mfr P/N" "0603WAF1822T5E"
 			(at 95.25 95.25 0)
 			(effects
@@
 			)
 		)
-		(property "Supplier_1 P/N" "C22793"
+		(property "Supplier_1 P/N" "C22892"
 			(at 95.25 95.25 0)
 			(effects
